Commit message: Release/2.1.0

File: tmc_gazebo_worlds/worlds/apartment.world.xacro (robot description, xacro)
@@ -12,5 +12,5 @@
       <pose>0 0 0 0 -0 0</pose>
       <link name='body'>
-        <pose>0 0 0 0 -0 0</pose>
+        <pose>5.0375 6.59 0 0 -0 0</pose>
         <collision name='gplane_coll'>
           <geometry>
@@ -43,9 +43,16 @@
           </geometry>
           <material>
-            <script>
-              <uri>model://base_materials/carpet/scripts</uri>
-              <uri>model://base_materials/carpet/textures</uri>
-              <name>carpet/carpet01</name>
-            </script>
+            <name>carpet</name>
+            <ambient>1 1 1 1</ambient>
+            <diffuse>0.5 0.5 0.5 1.0</diffuse>
+            <specular>0 0 0 1.0</specular>
+            <shininess>12.5</shininess>
+            <pbr>
+              <metal>
+                <albedo_map>../models/base_materials/carpet/textures/carpet01.png</albedo_map>
+                <max_anisotropy>16</max_anisotropy>
+                <scale>0.1 0.1</scale>
+              </metal>
+            </pbr>
           </material>
           <cast_shadows>0</cast_shadows>

File: tmc_gazebo_worlds/worlds/apartment_no_objects.world.xacro (robot description, xacro)
@@ -12,5 +12,5 @@
       <pose>0 0 0 0 -0 0</pose>
       <link name='body'>
-        <pose>0 0 0 0 -0 0</pose>
+        <pose>5.0375 6.59 0 0 -0 0</pose>
         <collision name='gplane_coll'>
           <geometry>
@@ -43,9 +43,16 @@
           </geometry>
           <material>
-            <script>
-              <uri>model://base_materials/carpet/scripts</uri>
-              <uri>model://base_materials/carpet/textures</uri>
-              <name>carpet/carpet01</name>
-            </script>
+            <name>carpet</name>
+            <ambient>1 1 1 1</ambient>
+            <diffuse>0.5 0.5 0.5 1.0</diffuse>
+            <specular>0 0 0 1.0</specular>
+            <shininess>12.5</shininess>
+            <pbr>
+              <metal>
+                <albedo_map>../models/base_materials/carpet/textures/carpet01.png</albedo_map>
+                <max_anisotropy>16</max_anisotropy>
+                <scale>0.1 0.1</scale>
+              </metal>
+            </pbr>
           </material>
           <cast_shadows>0</cast_shadows>
@@ -116,5 +123,5 @@
       <static>1</static>
       <pose>-0.0275 -0.0275 0 0 0 0</pose>
-      <uri>model://wall_frame_55_55_2090_none_collision</uri>
+      <uri>../models/wall_frame_55_55_2090_none_collision</uri>
       <name>wall_x00y00</name>
     </include>
@@ -122,5 +129,5 @@
       <static>1</static>
       <pose>-0.0275 0.45 0 0 0 0</pose>
-      <uri>model://full_wall_55_900_2090_none_collision</uri>
+      <uri>../models/full_wall_55_900_2090_none_collision</uri>
       <name>wall_x00y01</name>
     </include>
@@ -128,5 +135,5 @@
       <static>1</static>
       <pose>-0.0275 1.35 0 0 0 0</pose>
-      <uri>model://half_glass_wall_55_900_2090_none_collision</uri>
+      <uri>../models/half_glass_wall_55_900_2090_none_collision</uri>
       <name>wall_x00y02</name>
     </include>
@@ -134,5 +141,5 @@
       <static>1</static>
       <pose>-0.0275 2.25 0 0 0 0</pose>
-      <uri>model://half_glass_wall_55_900_2090_none_collision</uri>
+      <uri>../models/half_glass_wall_55_900_2090_none_collision</uri>
       <name>wall_x00y03</name>
     </include>
@@ -140,5 +147,5 @@
       <static>1</static>
       <pose>-0.0275 3.15 0 0 0 0</pose>
-      <uri>model://half_glass_wall_55_900_2090_none_collision</uri>
+      <uri>../models/half_glass_wall_55_900_2090_none_collision</uri>
       <name>wall_x00y04</name>
     </include>
@@ -146,5 +153,5 @@
       <static>1</static>
       <pose>-0.0275 4.05 0 0 0 0</pose>
-      <uri>model://full_wall_55_900_2090_none_collision</uri>
+      <uri>../models/full_wall_55_900_2090_none_collision</uri>
       <name>wall_x00y05</name>
     </include>
@@ -152,5 +159,5 @@
       <static>1</static>
       <pose>-0.0275 4.95 0 0 0 0</pose>
-      <uri>model://half_glass_wall_55_900_2090_none_collision</uri>
+      <uri>../models/half_glass_wall_55_900_2090_none_collision</uri>
       <name>wall_x00y06</name>
     </include>
@@ -158,5 +165,5 @@
       <static>1</static>
       <pose>-0.0275 5.85 0 0 0 0</pose>
-      <uri>model://half_glass_wall_55_900_2090_none_collision</uri>
+      <uri>../models/half_glass_wall_55_900_2090_none_collision</uri>
       <name>wall_x00y07</name>
     </include>
@@ -164,5 +171,5 @@
       <static>1</static>
       <pose>-0.0275 6.75 0 0 0 0</pose>
-      <uri>model://half_glass_wall_55_900_2090_none_collision</uri>
+      <uri>../models/half_glass_wall_55_900_2090_none_collision</uri>
       <name>wall_x00y08</name>
     </include>
@@ -170,5 +177,5 @@
       <static>1</static>
       <pose>-0.0275 7.65 0 0 0 0</pose>
-      <uri>model://full_wall_55_900_2090_none_collision</uri>
+      <uri>../models/full_wall_55_900_2090_none_collision</uri>
       <name>wall_x00y09</name>
     </include>
@@ -176,5 +183,5 @@
       <static>1</static>
       <pose>-0.0275 8.55 0 0 0 0</pose>
-      <uri>model://full_wall_55_900_2090_none_collision</uri>
+      <uri>../models/full_wall_55_900_2090_none_collision</uri>
       <name>wall_x00y10</name>
     </include>
@@ -182,5 +189,5 @@
       <static>1</static>
       <pose>-0.0275 9.45 0 0 0 0</pose>
-      <uri>model://full_wall_55_900_2090_none_collision</uri>
+      <uri>../models/full_wall_55_900_2090_none_collision</uri>
       <name>wall_x00y11</name>
     </include>
@@ -188,5 +195,5 @@
       <static>1</static>
       <pose>-0.0275 10.35 0 0 0 0</pose>
-      <uri>model://full_wall_55_900_2090_none_collision</uri>
+      <uri>../models/full_wall_55_900_2090_none_collision</uri>
       <name>wall_x00y12</name>
     </include>
@@ -194,5 +201,5 @@
       <static>1</static>
       <pose>-0.0275 11.25 0 0 0 0</pose>
-      <uri>model://half_glass_wall_55_900_2090_none_collision</uri>
+      <uri>../models/half_glass_wall_55_900_2090_none_collision</uri>
       <name>wall_x00y13</name>
     </include>
@@ -200,5 +207,5 @@
       <static>1</static>
       <pose>-0.0275 12.15 0 0 0 0</pose>
-      <uri>model://full_wall_55_900_2090_none_collision</uri>
+      <uri>../models/full_wall_55_900_2090_none_collision</uri>
       <name>wall_x00y14</name>
     </include>
@@ -206,5 +213,5 @@
       <static>1</static>
       <pose>-0.0275 12.73 0 0 0 0</pose>
-      <uri>model://full_wall_55_900_2090_none_collision</uri>
+      <uri>../models/full_wall_55_900_2090_none_collision</uri>
       <name>wall_x00y15</name>
     </include>
@@ -212,5 +219,5 @@
       <static>1</static>
       <pose>-0.0275 13.2075 0 0 0 0</pose>
-      <uri>model://wall_frame_55_55_2090_none_collision</uri>
+      <uri>../models/wall_frame_55_55_2090_none_collision</uri>
       <name>wall_x00y16</name>
     </include>
@@ -218,5 +225,5 @@
       <static>1</static>
       <pose>0.45 -0.0275 0 0 0 1.5708</pose>
-      <uri>model://full_wall_55_900_2090_none_collision</uri>
+      <uri>../models/full_wall_55_900_2090_none_collision</uri>
       <name>wall_x01y00</name>
     </include>
@@ -224,5 +231,5 @@
       <static>1</static>
       <pose>1.35 -0.0275 0 0 0 1.5708</pose>
-      <uri>model://half_glass_wall_55_900_2090_none_collision</uri>
+      <uri>../models/half_glass_wall_55_900_2090_none_collision</uri>
       <name>wall_x02y00</name>
     </include>
@@ -230,5 +237,5 @@
       <static>1</static>
       <pose>2.25 -0.0275 0 0 0 1.5708</pose>
-      <uri>model://half_glass_wall_55_900_2090_none_collision</uri>
+      <uri>../models/half_glass_wall_55_900_2090_none_collision</uri>
       <name>wall_x03y00</name>
     </include>
@@ -236,5 +243,5 @@
       <static>1</static>
       <pose>3.15 -0.0275 0 0 0 1.5708</pose>
-      <uri>model://full_wall_55_900_2090_none_collision</uri>
+      <uri>../models/full_wall_55_900_2090_none_collision</uri>
       <name>wall_x04y00</name>
     </include>
@@ -242,5 +249,5 @@
       <static>1</static>
       <pose>4.05 -0.0275 0 0 0 1.5708</pose>
-      <uri>model://full_wall_55_900_2090_none_collision</uri>
+      <uri>../models/full_wall_55_900_2090_none_collision</uri>
       <name>wall_x05y00</name>
     </include>
@@ -248,5 +255,5 @@
       <static>1</static>
       <pose>4.95 -0.0275 0 0 0 1.5708</pose>
-      <uri>model://half_glass_wall_55_900_2090_none_collision</uri>
+      <uri>../models/half_glass_wall_55_900_2090_none_collision</uri>
       <name>wall_x06y00</name>
     </include>
@@ -254,5 +261,5 @@
       <static>1</static>
       <pose>5.85 -0.0275 0 0 0 1.5708</pose>
-      <uri>model://half_glass_wall_55_900_2090_none_collision</uri>
+      <uri>../models/half_glass_wall_55_900_2090_none_collision</uri>
       <name>wall_x07y00</name>
     </include>
@@ -260,5 +267,5 @@
       <static>1</static>
       <pose>6.75 -0.0275 0 0 0 1.5708</pose>
-      <uri>model://full_wall_55_900_2090_none_collision</uri>
+      <uri>../models/full_wall_55_900_2090_none_collision</uri>
       <name>wall_x08y00</name>
     </include>
@@ -266,5 +273,5 @@
       <static>1</static>
       <pose>7.65 -0.0275 0 0 0 1.5708</pose>
-      <uri>model://half_glass_wall_55_900_2090_none_collision</uri>
+      <uri>../models/half_glass_wall_55_900_2090_none_collision</uri>
       <name>wall_x09y00</name>
     </include>
@@ -272,5 +279,5 @@
       <static>1</static>
       <pose>8.55 -0.0275 0 0 0 1.5708</pose>
-      <uri>model://half_glass_wall_55_900_2090_none_collision</uri>
+      <uri>../models/half_glass_wall_55_900_2090_none_collision</uri>
       <name>wall_x10y00</name>
     </include>
@@ -278,5 +285,5 @@
       <static>1</static>
       <pose>9.45 -0.0275 0 0 0 1.5708</pose>
-      <uri>model://full_wall_55_900_2090_none_collision</uri>
+      <uri>../models/full_wall_55_900_2090_none_collision</uri>
       <name>wall_x11y00</name>
     </include>
@@ -284,5 +291,5 @@
       <static>1</static>
       <pose>9.625 -0.0275 0 0 0 1.5708</pose>
-      <uri>model://full_wall_55_900_2090_none_collision</uri>
+      <uri>../models/full_wall_55_900_2090_none_collision</uri>
       <name>wall_x12y00</name>
     </include>
@@ -290,5 +297,5 @@
       <static>1</static>
       <pose>10.1025 -0.0275 0 0 0 0</pose>
-      <uri>model://wall_frame_55_55_2090_none_collision</uri>
+      <uri>../models/wall_frame_55_55_2090_none_collision</uri>
       <name>wall_x13y00</name>
     </include>
@@ -296,5 +303,5 @@
       <static>1</static>
       <pose>10.1025 0.45 0 0 0 0</pose>
-      <uri>model://full_wall_55_900_2090_none_collision</uri>
+      <uri>../models/full_wall_55_900_2090_none_collision</uri>
       <name>wall_x13y01</name>
     </include>
@@ -302,5 +309,5 @@
       <static>1</static>
       <pose>10.1025 1.35 0 0 0 0</pose>
-      <uri>model://half_glass_wall_55_900_2090_none_collision</uri>
+      <uri>../models/half_glass_wall_55_900_2090_none_collision</uri>
       <name>wall_x13y02</name>
     </include>
@@ -308,5 +315,5 @@
       <static>1</static>
       <pose>10.1025 2.25 0 0 0 0</pose>
-      <uri>model://half_glass_wall_55_900_2090_none_collision</uri>
+      <uri>../models/half_glass_wall_55_900_2090_none_collision</uri>
       <name>wall_x13y03</name>
     </include>
@@ -314,5 +321,5 @@
       <static>1</static>
       <pose>10.1025 3.15 0 0 0 0</pose>
-      <uri>model://full_wall_55_900_2090_none_collision</uri>
+      <uri>../models/full_wall_55_900_2090_none_collision</uri>
       <name>wall_x13y04</name>
     </include>
@@ -320,5 +327,5 @@
       <static>1</static>
       <pose>10.1025 4.05 0 0 0 0</pose>
-      <uri>model://half_glass_wall_55_900_2090_none_collision</uri>
+      <uri>../models/half_glass_wall_55_900_2090_none_collision</uri>
       <name>wall_x13y05</name>
     </include>
@@ -326,5 +333,5 @@
       <static>1</static>
       <pose>10.1025 4.95 0 0 0 0</pose>
-      <uri>model://half_glass_wall_55_900_2090_none_collision</uri>
+      <uri>../models/half_glass_wall_55_900_2090_none_collision</uri>
       <name>wall_x13y06</name>
     </include>
@@ -332,5 +339,5 @@
       <static>1</static>
       <pose>10.1025 5.85 0 0 0 0</pose>
-      <uri>model://full_wall_55_900_2090_none_collision</uri>
+      <uri>../models/full_wall_55_900_2090_none_collision</uri>
       <name>wall_x13y07</name>
     </include>
@@ -338,5 +345,5 @@
       <static>1</static>
       <pose>10.1025 6.75 0 0 0 0</pose>
-      <uri>model://half_glass_wall_55_900_2090_none_collision</uri>
+      <uri>../models/half_glass_wall_55_900_2090_none_collision</uri>
       <name>wall_x13y08</name>
     </include>
@@ -344,5 +351,5 @@
       <static>1</static>
       <pose>10.1025 7.65 0 0 0 0</pose>
-      <uri>model://half_glass_wall_55_900_2090_none_collision</uri>
+      <uri>../models/half_glass_wall_55_900_2090_none_collision</uri>
       <name>wall_x13y09</name>
     </include>
@@ -350,5 +357,5 @@
       <static>1</static>
       <pose>10.1025 8.55 0 0 0 0</pose>
-      <uri>model://full_wall_55_900_2090_none_collision</uri>
+      <uri>../models/full_wall_55_900_2090_none_collision</uri>
       <name>wall_x13y10</name>
     </include>
@@ -356,5 +363,5 @@
       <static>1</static>
       <pose>10.1025 9.45 0 0 0 0</pose>
-      <uri>model://full_wall_55_900_2090_none_collision</uri>
+      <uri>../models/full_wall_55_900_2090_none_collision</uri>
       <name>wall_x13y11</name>
     </include>
@@ -362,5 +369,5 @@
       <static>1</static>
       <pose>10.1025 10.35 0 0 0 0</pose>
-      <uri>model://half_glass_wall_55_900_2090_none_collision</uri>
+      <uri>../models/half_glass_wall_55_900_2090_none_collision</uri>
       <name>wall_x13y12</name>
     </include>
@@ -368,5 +375,5 @@
       <static>1</static>
       <pose>10.1025 12.15 0 0 0 0</pose>
-      <uri>model://full_wall_55_900_2090_none_collision</uri>
+      <uri>../models/full_wall_55_900_2090_none_collision</uri>
       <name>wall_x13y14</name>
     </include>
@@ -374,5 +381,5 @@
       <static>1</static>
       <pose>10.1025 12.73 0 0 0 0</pose>
-      <uri>model://full_wall_55_900_2090_none_collision</uri>
+      <uri>../models/full_wall_55_900_2090_none_collision</uri>
       <name>wall_x13y15</name>
     </include>
@@ -380,5 +387,5 @@
       <static>1</static>
       <pose>10.1025 13.2075 0 0 0 0</pose>
-      <uri>model://wall_frame_55_55_2090_none_collision</uri>
+      <uri>../models/wall_frame_55_55_2090_none_collision</uri>
       <name>wall_x13y16</name>
     </include>
@@ -386,5 +393,5 @@
       <static>1</static>
       <pose>0.45 13.2075 0 0 0 1.5708</pose>
-      <uri>model://full_wall_55_900_2090_none_collision</uri>
+      <uri>../models/full_wall_55_900_2090_none_collision</uri>
       <name>wall_x01y16</name>
     </include>
@@ -392,5 +399,5 @@
       <static>1</static>
       <pose>2.25 13.2075 0 0 0 1.5708</pose>
-      <uri>model://full_wall_55_900_2090_none_collision</uri>
+      <uri>../models/full_wall_55_900_2090_none_collision</uri>
       <name>wall_x03y16</name>
     </include>
@@ -398,5 +405,5 @@
       <static>1</static>
       <pose>3.15 13.2075 0 0 0 1.5708</pose>
-      <uri>model://full_wall_55_900_2090_none_collision</uri>
+      <uri>../models/full_wall_55_900_2090_none_collision</uri>
       <name>wall_x04y16</name>
     </include>
@@ -404,5 +411,5 @@
       <static>1</static>
       <pose>4.05 13.2075 0 0 0 1.5708</pose>
-      <uri>model://full_wall_55_900_2090_none_collision</uri>
+      <uri>../models/full_wall_55_900_2090_none_collision</uri>
       <name>wall_x05y16</name>
     </include>
@@ -410,5 +417,5 @@
       <static>1</static>
       <pose>4.95 13.2075 0 0 0 1.5708</pose>
-      <uri>model://full_wall_55_900_2090_none_collision</uri>
+      <uri>../models/full_wall_55_900_2090_none_collision</uri>
       <name>wall_x06y16</name>
     </include>
@@ -416,5 +423,5 @@
       <static>1</static>
       <pose>5.85 13.2075 0 0 0 1.5708</pose>
-      <uri>model://full_wall_55_900_2090_none_collision</uri>
+      <uri>../models/full_wall_55_900_2090_none_collision</uri>
       <name>wall_x07y16</name>
     </include>
@@ -422,5 +429,5 @@
       <static>1</static>
       <pose>6.75 13.2075 0 0 0 1.5708</pose>
-      <uri>model://full_wall_55_900_2090_none_collision</uri>
+      <uri>../models/full_wall_55_900_2090_none_collision</uri>
       <name>wall_x08y16</name>
     </include>
@@ -428,5 +435,5 @@
       <static>1</static>
       <pose>7.65 13.2075 0 0 0 1.5708</pose>
-      <uri>model://half_glass_wall_55_900_2090_none_collision</uri>
+      <uri>../models/half_glass_wall_55_900_2090_none_collision</uri>
       <name>wall_x09y16</name>
     </include>
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
File: tmc_gazebo_worlds/worlds/empty.world.xacro (robot description, xacro)
@@ -6,10 +6,42 @@
         <shadows>0</shadows>
     </scene>
-    <include>
-      <uri>model://sun</uri>
-    </include>
-    <include>
-      <uri>model://ground_plane</uri>
-    </include>
+    <light name="sun" type="directional">
+      <cast_shadows>true</cast_shadows>
+      <pose>0 0 10 0 0 0</pose>
+      <diffuse>0.8 0.8 0.8 1</diffuse>
+      <specular>0.2 0.2 0.2 1</specular>
+      <attenuation>
+        <range>1000</range>
+        <constant>0.9</constant>
+        <linear>0.01</linear>
+        <quadratic>0.001</quadratic>
+      </attenuation>
+      <direction>-0.5 0.1 -0.9</direction>
+    </light>
+    <model name="ground_plane">
+      <static>true</static>
+      <pose>0 0 0 0 0 0</pose>
+      <link name="link">
+        <collision name="collision">
+          <geometry>
+            <plane>
+              <size>20 20 0.1</size>
+            </plane>
+          </geometry>
+        </collision>
+        <visual name="visual">
+          <geometry>
+            <plane>
+              <size>20 20 0.1</size>
+            </plane>
+          </geometry>
+          <material>
+            <ambient>0.8 0.8 0.8 1</ambient>
+            <diffuse>0.8 0.8 0.8 1</diffuse>
+            <specular>0.8 0.8 0.8 1</specular>
+          </material>
+        </visual>
+      </link>
+    </model>
   </world>
 </sdf>

File: tmc_gazebo_worlds/worlds/hcr2013.world.xacro (robot description, xacro)
@@ -42,8 +42,14 @@
           </geometry>
           <material>
-            <script>
-              <uri>model://base_materials/wood/scripts/wood.material</uri>
-              <name>base_materials/hardwood_floor</name>
-            </script>
+            <name>hardwood_floor</name>
+            <diffuse>0.3 0.3 0.3 1.0</diffuse>
+            <pbr>
+              <metal>
+                <albedo_map>../models/base_materials/wood/textures/light_wood.png</albedo_map>
+                <max_anisotropy>16</max_anisotropy>
+                <rotate>90</rotate>
+                <scale>0.1 0.1</scale>
+              </metal>
+            </pbr>
           </material>
           <cast_shadows>0</cast_shadows>

File: tmc_gazebo_worlds/worlds/include/physics.xacro (robot description, xacro)
@@ -2,18 +2,31 @@
 <sdf version="1.4" xmlns:xacro="http://www.ros.org/wiki/xacro">
   <xacro:arg name="fast_physics" default="true" />
-  <physics type="ode">
-    <xacro:if value="$(arg fast_physics)">
-    <real_time_update_rate>333.0</real_time_update_rate>
-    <max_step_size>0.003</max_step_size>
-    <ode>
-      <solver>
-        <type>quick</type>
-        <iters>100</iters>
-      </solver>
-      <constraints>
-        <cfm>0.0001</cfm>
-      </constraints>
-    </ode>
-    </xacro:if>
-  </physics>
+  <plugin filename="gz-sim-physics-system" name="gz::sim::systems::Physics"/>
+  <plugin filename="gz-sim-user-commands-system" name="gz::sim::systems::UserCommands"/>
+  <plugin filename="gz-sim-scene-broadcaster-system" name="gz::sim::systems::SceneBroadcaster"/>
+  <plugin filename="gz-sim-sensors-system" name="gz::sim::systems::Sensors"/>
+  <plugin filename="gz-sim-imu-system" name="gz::sim::systems::Imu"/>
+  <plugin filename="ignition-gazebo-forcetorque-system" name="ignition::gazebo::systems::ForceTorque"/>
+  <gravity>0 0 -9.8</gravity>
+  <xacro:if value="$(arg fast_physics)">
+    <physics type="ode">
+      <real_time_update_rate>333.0</real_time_update_rate>
+      <max_step_size>0.003</max_step_size>
+      <ode>
+        <solver>
+          <type>quick</type>
+          <iters>100</iters>
+        </solver>
+        <constraints>
+          <cfm>0.0001</cfm>
+        </constraints>
+      </ode>
+    </physics>
+  </xacro:if>
+  <xacro:unless value="$(arg fast_physics)">
+    <physics name="1ms" type="ignored">
+      <max_step_size>0.005</max_step_size>
+      <real_time_factor>1.0</real_time_factor>
+    </physics>
+  </xacro:unless>
 </sdf>

File: tmc_gazebo_worlds/worlds/megaweb2015_no_objects.world.xacro (robot description, xacro)
@@ -12,7 +12,29 @@
       </camera>
     </gui>
-    <include>
-      <uri>model://ground_plane</uri>
-    </include>
+    <model name="ground_plane">
+      <static>true</static>
+      <pose>0 0 0 0 0 0</pose>
+      <link name="link">
+        <collision name="collision">
+          <geometry>
+            <plane>
+              <size>100 100 0.1</size>
+            </plane>
+          </geometry>
+        </collision>
+        <visual name="visual">
+          <geometry>
+            <plane>
+              <size>100 100 0.1</size>
+            </plane>
+          </geometry>
+          <material>
+            <ambient>0.8 0.8 0.8 1</ambient>
+            <diffuse>0.8 0.8 0.8 1</diffuse>
+            <specular>0.8 0.8 0.8 1</specular>
+          </material>
+        </visual>
+      </link>
+    </model>
     <light name='floorlight1' type='spot'>
       <cast_shadows>true</cast_shadows>

File: tmc_gazebo_worlds/worlds/mock_home.world.xacro (robot description, xacro)
@@ -42,9 +42,16 @@
           </geometry>
           <material>
-            <script>
-              <uri>model://base_materials/carpet/scripts</uri>
-              <uri>model://base_materials/carpet/textures</uri>
-              <name>carpet/carpet01</name>
-            </script>
+            <name>carpet</name>
+            <ambient>1 1 1 1</ambient>
+            <diffuse>0.5 0.5 0.5 1.0</diffuse>
+            <specular>0 0 0 1.0</specular>
+            <shininess>12.5</shininess>
+            <pbr>
+              <metal>
+                <albedo_map>../models/base_materials/carpet/textures/carpet01.png</albedo_map>
+                <max_anisotropy>16</max_anisotropy>
+                <scale>0.1 0.1</scale>
+              </metal>
+            </pbr>
           </material>
           <cast_shadows>0</cast_shadows>
